File: JBC-T245/JBC-Lötkolbenmodul.sch (KiCad schematic (older format))
At the start: 78 parts, among them IC101 ATMEGA328P-A, IC102 SP3485EN, IC103 INA193, IC104 CNY17-1, K101 XLR5, K102 Lötkolben_1_CONN_3, P101 CONN_01X03, P102 CONN_3X2, P103 2 externe Pins, P104 CONN_01X01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

Commit message: schutz für den Temperaturmesswandler verbessert
Parts:
- R117, R118: value 470 -> 5,6k
Other:
- note added: "Maximalspannung 1,25V am ADC,\nmaximal 25mV am Kolben (600°C)\nheißt: Gain = 44 (hier dann 50)"
- note removed: "Maximalspannung 1,1V am ADC,\nmaximal 25mV am Kolben (600°C)\nheißt: Gain = 44 (hier dann 50)"
- note removed: "hier Temp-Messerverstärker mit INA331"
